Commit message: basic simulated robot

File: protobot_description/urdf/gazebo.xacro (robot description, xacro)
@@ -1,12 +1,12 @@
 <?xml version="1.0"?>
 <robot xmlns:xacro="http://www.ros.org/wiki/xacro">
-    <gazebo>
+    <!-- <gazebo>
         <plugin
             filename="gz-sim-joint-state-publisher-system"
             name="gz::sim::systems::JointStatePublisher">
             <topic>joint_states</topic>
-            <joint_name>joint1</joint_name>
-            <joint_name>joint2</joint_name>
-            <joint_name>joint3</joint_name>
+            <joint_name>shoulder_joint</joint_name>
+            <joint_name>elbow_joint</joint_name>
+            <joint_name>wrist_joint</joint_name>
         </plugin>
     </gazebo>
@@ -15,5 +15,5 @@
             filename="gz-sim-joint-position-controller-system"
             name="gz::sim::systems::JointPositionController">
-            <joint_name>joint1</joint_name>
+            <joint_name>shoulder_joint</joint_name>
             <p_gain>1</p_gain>
             <i_gain>0.1</i_gain>
@@ -23,5 +23,5 @@
             filename="gz-sim-joint-position-controller-system"
             name="gz::sim::systems::JointPositionController">
-            <joint_name>joint2</joint_name>
+            <joint_name>elbow_joint</joint_name>
             <p_gain>1</p_gain>
             <i_gain>0.1</i_gain>
@@ -31,5 +31,5 @@
             filename="gz-sim-joint-position-controller-system"
             name="gz::sim::systems::JointPositionController">
-            <joint_name>joint3</joint_name>
+            <joint_name>wrist_joint</joint_name>
             <p_gain>1</p_gain>
             <i_gain>0.1</i_gain>
@@ -56,9 +56,9 @@
             <topic>rgb_camera/image_raw</topic>
         </sensor>
+    </gazebo> -->
+    <gazebo>
+        <plugin filename="gz_ros2_control-system" name="gz_ros2_control::GazeboSimROS2ControlPlugin">
+            <parameters>$(find protobot_controller)/config/controllers.yaml</parameters>
+        </plugin>
     </gazebo>
-    <!-- <gazebo>
-        <plugin filename="gz_ros2_control-system" name="gz_ros2_control::GazeboSimROS2ControlPlugin">
-            <parameters>$(find protobot_controller)/config/protobot_controllers.yaml</parameters>
-        </plugin>
-    </gazebo> -->
 </robot>

File: protobot_description/urdf/protobot.urdf.xacro (robot description, xacro)
@@ -1,6 +1,8 @@
 <?xml version="1.0"?>
-<robot name="arduinobot" xmlns:xacro="http://www.ros.org/wiki/xacro">
+<robot name="protobot" xmlns:xacro="http://www.ros.org/wiki/xacro">
+    <xacro:arg name="is_sim" default="true"/>
     <xacro:include filename="$(find protobot_description)/urdf/common_properties.xacro"/>
     <xacro:include filename="$(find protobot_description)/urdf/structure.xacro"/>
     <xacro:include filename="$(find protobot_description)/urdf/gazebo.xacro"/>
+    <xacro:include filename="$(find protobot_description)/urdf/controls.xacro"/>
 </robot>

File: protobot_description/urdf/structure.xacro (robot description, xacro)
@@ -253,5 +253,5 @@
         <child link="rod1_link" />
     </joint>
-    <joint name="joint1" type="revolute">
+    <joint name="shoulder_joint" type="revolute">
         <origin xyz="0.075 0 0.025" rpy="0 0 0" />
         <parent link="rod1_link" />
@@ -270,5 +270,5 @@
         <child link="servo2_link" />
     </joint>
-    <joint name="joint2" type="revolute">
+    <joint name="elbow_joint" type="revolute">
         <origin xyz="0.03 0 0.025" rpy="0 0 0" />
         <parent link="servo2_link" />
@@ -282,5 +282,5 @@
         <child link="servo3_link" />
     </joint>
-    <joint name="joint3" type="revolute">
+    <joint name="wrist_joint" type="revolute">
         <origin xyz="0.03 0 0.025" rpy="0 0 0" />
         <parent link="servo3_link" />

Commit message: adding kinematics

File: protobot_description/urdf/gazebo.xacro (robot description, xacro)
@@ -57,4 +57,34 @@
         </sensor>
     </gazebo> -->
+    <gazebo reference="camera_link">
+        <sensor name="camera" type="camera">
+            <camera>
+                <horizontal_fov>1.3962634</horizontal_fov>
+                <image>
+                    <width>640</width>
+                    <height>480</height>
+                    <format>R8G8B8</format>
+                </image>
+                <clip>
+                    <near>0.1</near>
+                    <far>15</far>
+                </clip>
+                <noise>
+                    <type>gaussian</type>
+                        <!-- Noise is sampled independently per pixel on each frame.
+                            That pixel's noise value is added to each of its color
+                            channels, which at that point lie in the range [0,1]. -->
+                    <mean>0.0</mean>
+                    <stddev>0.007</stddev>
+                </noise>
+                <optical_frame_id>camera_link_optical</optical_frame_id>
+                <camera_info_topic>arm_camera/camera_info</camera_info_topic>
+            </camera>
+            <always_on>1</always_on>
+            <update_rate>20</update_rate>
+            <visualize>true</visualize>
+            <topic>arm_camera/image</topic>
+        </sensor>
+    </gazebo>
     <gazebo>
         <plugin filename="gz_ros2_control-system" name="gz_ros2_control::GazeboSimROS2ControlPlugin">

File: protobot_description/urdf/structure.xacro (robot description, xacro)
@@ -238,4 +238,6 @@
         </inertial>
     </link>
+    <link name="camera_link_optical">
+    </link>
     <joint name="world_base_joint" type="fixed">
         <origin xyz="0 0 0" rpy="0 0 0" />
@@ -294,3 +296,8 @@
         <child link="camera_link" />
     </joint>
+    <joint name="camera_optical_joint" type="fixed">
+        <origin xyz="0.005 0.02 0.01" rpy="-1.5707 0 -1.5707"/>
+        <parent link="camera_link"/>
+        <child link="camera_link_optical"/>
+    </joint>
 </robot>
